Commit message: Update my_robot.urdf

File: my_robot.urdf (robot description, URDF)
Before this commit: robot my_robot, 2 links, 1 joints
Links:
- added link third_link; visual box size=0.4 0.3 0.1
- link base_link: geometry visual box size=0.8 0.3 0.2
- link second_link: geometry visual box size=0.8 0.3 0.2
Joints:
- removed joint base_second_joint
- added joint ankle_joint: type fixed, parent second_link, child third_link, origin xyz=0.8 0 0 rpy=0 -1.14 0
- added joint knee_joint: type fixed, parent base_link, child second_link, origin xyz=0.8 0 0 rpy=0 0.57 0
